File: hex-dna.kicad_pcb (KiCad board)
At the start: 2 copper layers, 79.5 x 69 mm, 21 parts, among them J1 +5V GND, J2 LED1 VCC GND, J3 LED2 GND VCC, J4 LED3 GND VCC, J7 LED4 GND VCC

Commit message: fixed minor silkscreen error
Parts:
- J2: value LED1 VCC GND -> LED1 GND VCC
Changed lines of the file:
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@@
 			)
 		)
-		(property "Value" "LED1 VCC GND"
+		(property "Value" "LED1 GND VCC"
 			(at 2.5 2.5 0)
 			(layer "F.SilkS")
